Commit message: controlbox mesh added

File: urdf/inc/ur_controlbox.urdf.xacro (robot description, xacro)
@@ -16,5 +16,5 @@
         <origin xyz="0 0 0" rpy="0 0 0"/>
         <geometry>
-          <mesh filename="file://$(find ur_description)/meshes/common/simplify_control-box.stl" scale="0.001 0.001 0.001" />
+          <mesh filename="file://$(find ur_description)/meshes/common/control-box-simplified.stl" scale="0.001 0.001 0.001" />
         </geometry>
         <!-- <material name="plastic"/> -->
@@ -23,5 +23,5 @@
         <origin xyz="0 0 0" rpy="0 0 0"/>
         <geometry>
-          <mesh filename="file://$(find ur_description)/meshes/common/simplify_control-box.stl" scale="0.001 0.001 0.001" />
+          <mesh filename="file://$(find ur_description)/meshes/common/control-box-simplified.stl" scale="0.001 0.001 0.001" />
         </geometry>
       </collision>
